File: Input.kicad_sch (KiCad schematic)
At the start: 8 parts, among them SW1 SW_Push, SW2 SW_Push, SW3 SW_Push, SW4 SW_Push, SW5 SW_Push, SW6 SW_Push, SW7 SW_Push, SW8 SW_Push

Commit message: slight updates
Connections:
- no-connect marks 0 -> 8
Changed lines of the file:
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@@
   (junction (at 121.92 68.58) (diameter 0) (color 0 0 0 0)
   )
+  (no_connect (at 53.34 50.8))
+  (no_connect (at 111.76 57.15))
+  (no_connect (at 53.34 87.63))
+  (no_connect (at 53.34 76.2))
+  (no_connect (at 86.36 57.15))
+  (no_connect (at 53.34 63.5))
+  (no_connect (at 111.76 68.58))
+  (no_connect (at 86.36 68.58))
   (wire (pts (xy 96.52 57.15) (xy 96.52 68.58))
     (stroke (width 0) (type default))
