File: Page_1.kicad_sch (KiCad schematic)
At the start: 9 parts, among them U3 DDR2_SODIMM_CM_3_Lite, U4 1040310811

Commit message: slight updates
Connections:
- net CM_3V3: now also C18.1, U4.4 (VDD)
- net 3V3 renamed +3V3
- net +3V3: no longer C18.1, U4.4 (VDD)
- no-connect marks 66 -> 87
Other:
- moved on the sheet: R3, R4, R5
