File: PiCM3_GBA.kicad_pcb (KiCad board)
At the start: 4 copper layers, 130.7 x 72.9 mm, 48 parts, among them J1 Conn_01x02_Shielded, P1 USB_C_Plug_USB2.0, U1 PAM2306AYPKE, U2 MCP73871, U3 DDR2_SODIMM_CM_3_Lite, U4 1040310811

Commit message: slight updates
Parts:
- moved R12 15.7 mm to (156.5, 150.6), turned to -90 degrees
- moved R1 13.2 mm to (58.2, 128.8), turned to 0 degrees
- moved R14 11.4 mm to (165.1, 150.6), turned to 180 degrees
- moved R4 10.7 mm to (107.2, 128.5), turned to 180 degrees
- moved R10 10.7 mm to (167.4, 158.0)
- moved R11 8.95 mm to (156.2, 154.9), turned to -90 degrees
- moved R5 5.93 mm to (110.5, 128.8), turned to 0 degrees
- moved C12 5.24 mm to (160.8, 163.1)
- moved C9 5.24 mm to (160.8, 160.5)
- moved C4 4.92 mm to (55.9, 136.7)
- moved C5 1.22 mm to (55.8, 139.3)
Connections:
- net 1V8 renamed CM_1V8
- net 3V3 renamed CM_3V3
- net 5V renamed CM_VBAT
Routing:
- net VDDI: track 0.00 -> 41.1 mm
- net CM_3V3: track 0.00 -> 26.0 mm
- net Net-(J1-Pin_1): track 0.00 -> 14.3 mm, vias 0 -> 1
- net CM_1V8: track 0.00 -> 8.97 mm
- net Net-(U1-LX1): track 0.00 -> 7.60 mm
- net Net-(U2-VPCC): track 0.00 -> 6.82 mm
- net Net-(U5-CSX): track 0.00 -> 6.34 mm
- net Net-(U5-LEDA1): track 0.00 -> 5.69 mm
- net Net-(U1-LX2): track 0.00 -> 5.62 mm
- net Net-(U5-LEDA4): track 0.00 -> 5.34 mm
- net Net-(U5-LEDA2): track 0.00 -> 5.16 mm
- net Net-(U5-LEDA3): track 0.00 -> 4.91 mm
- net Net-(U1-EN2): track 0.00 -> 4.76 mm
- net CM_VBAT: track 0.00 -> 4.58 mm
- net Net-(P1-CC): track 0.00 -> 4.42 mm
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