File: Power.kicad_sch (KiCad schematic)
At the start: 34 parts, among them J1 Conn_01x02_Shielded, P1 USB_C_Plug_USB2.0, U1 PAM2306AYPKE, U2 MCP73871

Commit message: slight updates
Connections:
- net 1V8 renamed +1V8
- net 3V3 renamed +3V3
- net 5V renamed +5V
Other:
- moved on the sheet: C11, C13, C7, P1, R13
